File: pcb_boards/gateway/pcb_gateway.kicad_pcb (KiCad board)
At the start: 2 copper layers, 76 x 92.5 mm, 99 parts, among them IC1 PCF2129AT, J1 Micro_SD_Card, J2 USB_B_Micro, J3 Conn_02x03_Counter_Clockwise, J4 Conn_01x02, J5 Conn_01x02, Q1 S8050, Q2 S8050, SW1 SW_SPST, SW2 SW_Push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

Commit message: Update.
Parts:
- removed AE3: Conn_Coaxial, Connector_Coaxial:SMA_Amphenol_901-144_Vertical
- removed BT4: Battery_Cell, gems_footprints:Renata_Battery_Holder_SMTM1125
- removed C15, C19, C25, C5: 100nF, Capacitor_SMD:C_0603_1608Metric
- removed J1: Micro_SD_Card, Connector_Card:microSD_HC_Wuerth_693072010801
- removed R13, R14: 330R, Resistor_SMD:R_0603_1608Metric
- removed R5, R6: 10k, Resistor_SMD:R_0603_1608Metric
- removed U11: MTK3339, gems_footprints:FGPMMOPA6H
- removed U2: SiP32431, Package_TO_SOT_SMD:SOT-363_SC-70-6
- C2, C3, C4, C6, C7: footprint Capacitor_SMD:C_1206_3216Metric -> Capacitor_SMD:C_1210_3225Metric
- C27: value 100nF -> 1uF; moved to F.Cu
- H1: moved to B.Cu
- U7: value SHTC3 -> SiP32431; footprint gems_footprints:DFN_4_Pin_2x2mm -> Package_TO_SOT_SMD:SOT-363_SC-70-6
- moved U7 60.4 mm to (65.4, 67.4), turned to 180 degrees
- moved C26 46.0 mm to (65.4, 63.2), turned to 180 degrees
- moved C27 12.6 mm to (65.4, 69.8), turned to 0 degrees
- moved C20 10.6 mm to (84.6, 104.8), turned to 270 degrees
- moved C7 0.70 mm to (72.4, 95.5)
- moved L1 0.30 mm to (68.0, 93.7)
Connections:
- C10 pad 1: +4V -> /REG_4V
- C26 pad 2: +3V3 -> +4V
- C27 pad 2: VPP -> /REG_4V
- C29 pad 2: +4V -> /REG_4V
- U1 pad 12: /M_SEL1 -> /EN_GPRS
- U1 pad 14: /~CS_SD -> /DTR_SIM_LV
- U1 pad 23: /EN_BM -> Net-(U1-Pad23)
- U1 pad 24: /~RST_GPS -> Net-(U1-Pad24)
- U1 pad 26: /GPS_FIX -> /EN_BM
- U1 pad 29: /DTR_SIM_LV -> Net-(U1-Pad29)
- U1 pad 8: /EN_VPP -> Net-(U1-Pad8)
- U10 pad 3: +4V -> /REG_4V
- U12 pad 14: +4V -> /REG_4V
- U6 pad 1: /RX_GPS -> Net-(U6-Pad1)
- U6 pad 10: /M_SEL0 -> GND
- U6 pad 12: /TX_GPS -> Net-(U6-Pad12)
- U6 pad 9: /M_SEL1 -> /M_SEL0
- U7 pad 1: +3V3 -> /REG_4V
- U7 pad 2: /SCL -> GND
- U7 pad 3: /SDA -> /EN_GPRS
- U7 pad 4: GND -> +4V
- U8 pad 2: +4V -> /REG_4V
Routing:
- net /MOSI: track 195.9 -> 70.9 mm, vias 7 -> 0
- net VPP: track 116.7 -> 0.00 mm, vias 7 -> 0
- net /REG_4V: track 0.00 -> 104.7 mm, vias 0 -> 5
- net /SCLK: track 142.9 -> 41.5 mm, vias 8 -> 2
- net /MISO: track 143.6 -> 46.5 mm, vias 9 -> 2
- net /EN_GPRS: track 0.00 -> 87.7 mm, vias 0 -> 2
- net /~CS_SD: track 80.9 -> 0.00 mm, vias 5 -> 0
- net /RX_GPS: track 54.7 -> 0.00 mm, vias 6 -> 0
- net +4V: track 145.4 -> 91.5 mm, vias 9 -> 6
- net /TX_GPS: track 48.3 -> 0.00 mm, vias 6 -> 0
- net /EN_VPP: track 45.9 -> 0.00 mm
- net /GPS_FIX: track 42.7 -> 0.00 mm, vias 2 -> 0
- net Net-(BT4-Pad1): track 30.3 -> 0.00 mm, vias 1 -> 0
- net GND: track 108.5 -> 79.7 mm, vias 137 -> 127
- net /~RST_GPS: track 27.0 -> 0.00 mm, vias 2 -> 0
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Other:
- board text added: "Rev. 3"
- board text removed: "Rev. 2"
