File: pcb_boards/sensor_node/sensor_node.kicad_pcb (KiCad board)
At the start: 2 copper layers, 93 x 93 mm, 61 parts, among them IC1 PCF2129AT, J2 Conn_02x03_Odd_Even, J3 USB_B_Micro, U1 SiP32431, U2 ESP32-WROOM-32, U3 RF-LORA-868-SO, U7 RP604x, U8 SiP32431

Commit message: Update.
Routing:
- net GND: vias 83 -> 86
Changed lines of the file:
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@@
 (kicad_pcb (version 20171130) (host pcbnew 5.1.5+dfsg1-2build2)
   (general
-    (thickness 1.6)
+    (thickness 0.8)
     (drawings 57)
-    (tracks 773)
+    (tracks 776)
     (zones 0)
     (modules 61)
@@
   (page A4)
   (layers
-    (0 F.Cu signal)
+    (0 F.Cu mixed)
     (31 B.Cu signal)
     (32 B.Adhes user)
@@
   )
   (setup
-    (last_trace_width 0.6)
+    (last_trace_width 0.25)
     (user_trace_width 0.25)
     (user_trace_width 0.3)
@@
     (user_trace_width 1)
     (trace_clearance 0.2)
-    (zone_clearance 0.25)
+    (zone_clearance 0.5)
     (zone_45_only yes)
     (trace_min 0.2)
@@
       (effects (font (size 1 1) (thickness 0.15)))
     )
-    (fp_line (start 0 -1.27) (end 3.81 -1.27) (layer F.Fab) (width 0.1))
-    (fp_line (start 3.81 -1.27) (end 3.81 6.35) (layer F.Fab) (width 0.1))
-    (fp_line (start 3.81 6.35) (end -1.27 6.35) (layer F.Fab) (width 0.1))
-    (fp_line (start -1.27 6.35) (end -1.27 0) (layer F.Fab) (width 0.1))
-    (fp_line (start -1.27 0) (end 0 -1.27) (layer F.Fab) (width 0.1))
-    (fp_line (start -1.33 6.41) (end 3.87 6.41) (layer F.SilkS) (width 0.12))
-    (fp_line (start -1.33 1.27) (end -1.33 6.41) (layer F.SilkS) (width 0.12))
-    (fp_line (start 3.87 -1.33) (end 3.87 6.41) (layer F.SilkS) (width 0.12))
-    (fp_line (start -1.33 1.27) (end 1.27 1.27) (layer F.SilkS) (width 0.12))
-    (fp_line (start 1.27 1.27) (end 1.27 -1.33) (layer F.SilkS) (width 0.12))
-    (fp_line (start 1.27 -1.33) (end 3.87 -1.33) (layer F.SilkS) (width 0.12))
-    (fp_line (start -1.33 0) (end -1.33 -1.33) (layer F.SilkS) (width 0.12))
-    (fp_line (start -1.33 -1.33) (end 0 -1.33) (layer F.SilkS) (width 0.12))
-    (fp_line (start -1.8 -1.8) (end -1.8 6.85) (layer F.CrtYd) (width 0.05))
-    (fp_line (start -1.8 6.85) (end 4.35 6.85) (layer F.CrtYd) (width 0.05))
-    (fp_line (start 4.35 6.85) (end 4.35 -1.8) (layer F.CrtYd) (width 0.05))
-    (fp_line (start 4.35 -1.8) (end -1.8 -1.8) (layer F.CrtYd) (width 0.05))
     (fp_text user %R (at 1.27 2.54) (layer F.Fab)
       (effects (font (size 1 1) (thickness 0.15)))
     )
-    (pad 1 thru_hole rect (at 0 0 90) (size 1.7 1.7) (drill 1) (layers *.Cu *.Mask)
-      (net 17 /TX))
-    (pad 2 thru_hole oval (at 2.54 0 90) (size 1.7 1.7) (drill 1) (layers *.Cu *.Mask)
-      (net 18 /RX))
-    (pad 3 thru_hole oval (at 0 2.54 90) (size 1.7 1.7) (drill 1) (layers *.Cu *.Mask)
-      (net 53 /~RST))
-    (pad 4 thru_hole oval (at 2.54 2.54 90) (size 1.7 1.7) (drill 1) (layers *.Cu *.Mask)
-      (net 54 /BOOT))
-    (pad 5 thru_hole oval (at 0 5.08 90) (size 1.7 1.7) (drill 1) (layers *.Cu *.Mask)
-      (net 1 GND))
+    (fp_line (start 4.35 -1.8) (end -1.8 -1.8) (layer F.CrtYd) (width 0.05))
+    (fp_line (start 4.35 6.85) (end 4.35 -1.8) (layer F.CrtYd) (width 0.05))
+    (fp_line (start -1.8 6.85) (end 4.35 6.85) (layer F.CrtYd) (width 0.05))
+    (fp_line (start -1.8 -1.8) (end -1.8 6.85) (layer F.CrtYd) (width 0.05))
+    (fp_line (start -1.33 -1.33) (end 0 -1.33) (layer F.SilkS) (width 0.12))
+    (fp_line (start -1.33 0) (end -1.33 -1.33) (layer F.SilkS) (width 0.12))
+    (fp_line (start 1.27 -1.33) (end 3.87 -1.33) (layer F.SilkS) (width 0.12))
+    (fp_line (start 1.27 1.27) (end 1.27 -1.33) (layer F.SilkS) (width 0.12))
+    (fp_line (start -1.33 1.27) (end 1.27 1.27) (layer F.SilkS) (width 0.12))
+    (fp_line (start 3.87 -1.33) (end 3.87 6.41) (layer F.SilkS) (width 0.12))
+    (fp_line (start -1.33 1.27) (end -1.33 6.41) (layer F.SilkS) (width 0.12))
+    (fp_line (start -1.33 6.41) (end 3.87 6.41) (layer F.SilkS) (width 0.12))
+    (fp_line (start -1.27 0) (end 0 -1.27) (layer F.Fab) (width 0.1))
+    (fp_line (start -1.27 6.35) (end -1.27 0) (layer F.Fab) (width 0.1))
+    (fp_line (start 3.81 6.35) (end -1.27 6.35) (layer F.Fab) (width 0.1))
+    (fp_line (start 3.81 -1.27) (end 3.81 6.35) (layer F.Fab) (width 0.1))
+    (fp_line (start 0 -1.27) (end 3.81 -1.27) (layer F.Fab) (width 0.1))
     (pad 6 thru_hole oval (at 2.54 5.08 90) (size 1.7 1.7) (drill 1) (layers *.Cu *.Mask)
       (net 1 GND))
+    (pad 5 thru_hole oval (at 0 5.08 90) (size 1.7 1.7) (drill 1) (layers *.Cu *.Mask)
+      (net 1 GND))
+    (pad 4 thru_hole oval (at 2.54 2.54 90) (size 1.7 1.7) (drill 1) (layers *.Cu *.Mask)
+      (net 54 /BOOT))
+    (pad 3 thru_hole oval (at 0 2.54 90) (size 1.7 1.7) (drill 1) (layers *.Cu *.Mask)
+      (net 53 /~RST))
+    (pad 2 thru_hole oval (at 2.54 0 90) (size 1.7 1.7) (drill 1) (layers *.Cu *.Mask)
+      (net 18 /RX))
+    (pad 1 thru_hole rect (at 0 0 90) (size 1.7 1.7) (drill 1) (layers *.Cu *.Mask)
+      (net 17 /TX))
     (model ${KISYS3DMOD}/Connector_PinHeader_2.54mm.3dshapes/PinHeader_2x03_P2.54mm_Vertical.wrl
       (at (xyz 0 0 0))
@@
     (fp_line (start 29 8.7) (end -29 8.7) (layer F.SilkS) (width 0.25))
     (fp_line (start -29 8.7) (end -29 -8.7) (layer F.SilkS) (width 0.25))
-    (fp_text user - (at 31 0 180) (layer F.SilkS)
+    (fp_text user - (at 31 0) (layer F.SilkS)
       (effects (font (size 3 3) (thickness 0.25)))
     )
-    (fp_text user + (at -31 0 180) (layer F.SilkS)
+    (fp_text user + (at -31 0) (layer F.SilkS)
       (effects (font (size 3 3) (thickness 0.25)))
     )
@@
     (fp_line (start 1.5 -1.35) (end 1.5 1.35) (layer F.CrtYd) (width 0.15))
     (fp_line (start -1.5 -1.35) (end 1.5 -1.35) (layer F.CrtYd) (width 0.15))
-    (pad 13 thru_hole circle (at 0 0 180) (size 0.75 0.75) (drill 0.5) (layers *.Cu *.Mask)
+    (pad 13 thru_hole circle (at 0 0 180) (size 1 1) (drill 0.4) (layers *.Cu *.Mask)
       (net 1 GND))
     (pad 13 smd rect (at 0 0 180) (size 2.5 1.5) (layers F.Cu F.Paste F.Mask)
@@
       (effects (font (size 1 1) (thickness 0.15)))
     )
-    (fp_line (start -3.5 -2.5) (end 3.5 -2.5) (layer F.CrtYd) (width 0.15))
-    (fp_line (start 3.5 -2.5) (end 3.5 2.5) (layer F.CrtYd) (width 0.15))
-    (fp_line (start 3.5 2.5) (end -3.5 2.5) (layer F.CrtYd) (width 0.15))
-    (fp_line (start -3.5 2.5) (end -3.5 -2.5) (layer F.CrtYd) (width 0.15))
-    (fp_line (start -0.7 -1.75) (end 0.7 -1.75) (layer F.Fab) (width 0.15))
-    (fp_line (start 0.7 -1.75) (end 2 -1) (layer F.Fab) (width 0.15))
-    (fp_line (start 2 -1) (end 2 1) (layer F.Fab) (width 0.15))
-    (fp_line (start 2 1) (end 0.7 1.75) (layer F.Fab) (width 0.15))
-    (fp_line (start 0.7 1.75) (end -0.7 1.75) (layer F.Fab) (width 0.15))
-    (fp_line (start -0.7 1.75) (end -2 1) (layer F.Fab) (width 0.15))
-    (fp_line (start -2 1) (end -2 -1) (layer F.Fab) (width 0.15))
     (fp_line (start -2 -1) (end -0.7 -1.75) (layer F.Fab) (width 0.15))
-    (pad 1 smd rect (at 1.55 0) (size 1.9 4) (layers F.Cu F.Paste F.Mask)
-      (net 22 "Net-(L1-Pad1)"))
+    (fp_line (start -2 1) (end -2 -1) (layer F.Fab) (width 0.15))
+    (fp_line (start -0.7 1.75) (end -2 1) (layer F.Fab) (width 0.15))
+    (fp_line (start 0.7 1.75) (end -0.7 1.75) (layer F.Fab) (width 0.15))
+    (fp_line (start 2 1) (end 0.7 1.75) (layer F.Fab) (width 0.15))
+    (fp_line (start 2 -1) (end 2 1) (layer F.Fab) (width 0.15))
+    (fp_line (start 0.7 -1.75) (end 2 -1) (layer F.Fab) (width 0.15))
+    (fp_line (start -0.7 -1.75) (end 0.7 -1.75) (layer F.Fab) (width 0.15))
+    (fp_line (start -3.5 2.5) (end -3.5 -2.5) (layer F.CrtYd) (width 0.15))
+    (fp_line (start 3.5 2.5) (end -3.5 2.5) (layer F.CrtYd) (width 0.15))
+    (fp_line (start 3.5 -2.5) (end 3.5 2.5) (layer F.CrtYd) (width 0.15))
+    (fp_line (start -3.5 -2.5) (end 3.5 -2.5) (layer F.CrtYd) (width 0.15))
     (pad 2 smd rect (at -1.55 0) (size 1.9 4) (layers F.Cu F.Paste F.Mask)
       (net 23 "Net-(L1-Pad2)"))
+    (pad 1 smd rect (at 1.55 0) (size 1.9 4) (layers F.Cu F.Paste F.Mask)
+      (net 22 "Net-(L1-Pad1)"))
   )
   (module gems_footprints:Renata_Battery_Holder_SMTM1125 (layer F.Cu)
@@
   (via (at 99.35 74.15) (size 0.8) (drill 0.4) (layers F.Cu B.Cu) (net 1))
   (via (at 96.6 56.35) (size 0.8) (drill 0.4) (layers F.Cu B.Cu) (net 1))
+  (via (at 110.55 80.2) (size 0.8) (drill 0.4) (layers F.Cu B.Cu) (net 1))
+  (via (at 114 80.2) (size 0.8) (drill 0.4) (layers F.Cu B.Cu) (net 1))
+  (via (at 84.65 75.45) (size 0.8) (drill 0.4) (layers F.Cu B.Cu) (net 1))
   (segment (start 83.2875 122.7125) (end 81.5 124.5) (width 1) (layer F.Cu) (net 2))
   (segment (start 83.2875 115.5) (end 83.2875 122.7125) (width 1) (layer F.Cu) (net 2))
@@
   (segment (start 63.5 64.8) (end 65.9 67.2) (width 0.35) (layer F.Cu) (net 71))
   (zone (net 1) (net_name GND) (layer F.Cu) (hatch edge 0.508)
-    (connect_pads (clearance 0.25))
+    (connect_pads (clearance 0.5))
     (min_thickness 0.254)
     (fill yes (arc_segments 16) (thermal_gap 0.508) (thermal_bridge_width 0.508))
@@
   )
   (zone (net 1) (net_name GND) (layer B.Cu) (hatch edge 0.508)
-    (connect_pads (clearance 0.25))
+    (connect_pads (clearance 0.5))
     (min_thickness 0.254)
     (fill yes (arc_segments 16) (thermal_gap 0.508) (thermal_bridge_width 0.508))
