File: pcb_boards/sensor_node/sensor_node.sch (KiCad schematic (older format))
At the start: 65 parts, among them IC1 PCF2129AT, J1 Conn_02x03_Counter_Clockwise, J2 Conn_01x02, J3 USB_B_Micro, J4 Conn_01x02, J5 Conn_01x02, U1 SiP32431, U2 ESP32-WROOM-32, U3 RF-LORA-868-SO, U5 SHTC3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

Commit message: Update.
Parts:
- AE1, H1, H2, H3, H4, H7: Price (none) -> 0
- ANT1: Price (none) -> 4.15
- BT1: Price (none) -> 0.529
- BT2: Mouser (none) -> 485-1769; Price (none) -> 0.635
- BT3: Mouser (none) -> Farnell 1365937; Price (none) -> 9.23
- C10, C15, C4, C5, C7, C9: Mouser (none) -> 810-CGA3E2X8R1E104K; Price (none) -> 0.136
- C11, C6: Mouser (none) -> 810-CGA5L1X7R1C685MC; Price (none) -> 0.364
- C13, C14, C17: Mouser (none) -> 963-TMK325BJ106KM-P; Price (none) -> 0.415
- C16, C18: Mouser (none) -> 963-TMK316BBJ226ML-T; Price (none) -> 0.449
- D2, D3, D4: Price (none) -> 0.36
- FB1: Price (none) -> 0.09
- I2C1, I2C2, I2C3: Mouser (none) -> Farnell: 1516281; Price (none) -> 0.138
- IC1: Mouser PCF2129T/2,518 -> 771-PCF2129T/2,518; Mouser Part Number 771-PCF2129T/2,518 -> (none); Price (none) -> 2.57
- IO2, IO3, OWI1, OWI2: Mouser (none) -> Farnell: 1516277; Price (none) -> 0.0968
- IO4, RESET1: Mouser Button_Switch_SMD:SW_SPST_KMR2 -> 611-KMR621NGLFS; Price (none) -> 0.33
- J1: Mouser (none) -> 571-5-146258-3; Price (none) -> 0.432
- J2, J4, J5: Mouser (none) -> 571-4-103328-1; Price (none) -> 0.212
- J3: Price (none) -> 0.70
- JP2: Mouser (none) -> 571-4-103321-5; Price (none) -> 0.237
- L1: Price (none) -> 0.169
- R1, R14, R15, R2, R4, R5, R8: Mouser (none) -> 284-APC0603B10K0N; Price (none) -> 0.102
- R10, R12: value R4.7k -> 4.7k; Mouser (none) -> 71-CRCW06034K70JNEAC; Price (none) -> 0.085
- R16, R7: Mouser (none) -> 603-RC0603FR-07750RL; Price (none) -> 0.085
- R3: Mouser (none) -> 603-RC0603JR-07330RL; Price (none) -> 0.085
- R9: Mouser (none) -> 71-CRCW060310M0FKEAC; Price (none) -> 0.085
- SPI1, SPI2: Mouser (none) -> Farnell: 1516282; Price (none) -> 0.151
- U1, U8: Price (none) -> 0.51
- U2: Price (none) -> 3.81
- U3: Mouser (none) -> Farnell: 2500100; Price (none) -> 17.11
- U5: Price (none) -> 2.07
- U7: Price (none) -> 1.8

Commit message: Update PCB.
Parts:
- added AE2: Antenna, RF_Antenna:Texas_SWRA416_868MHz_915MHz, symbol Device:Antenna
- added C1: 1pF, Capacitor_SMD:C_0603_1608Metric, symbol Device:C
- added JP1: Jumper_3_Open, Jumper:SolderJumper-3_P1.3mm_Open_Pad1.0x1.5mm, symbol Jumper:Jumper_3_Open
- added L2: 12nH, Inductor_SMD:L_0603_1608Metric, symbol Device:L
- I2C1: footprint Connector_JST:JST_XH_B05B-XH-A_1x05_P2.50mm_Vertical -> Connector_JST:JST_XH_B5B-XH-A_1x05_P2.50mm_Vertical
Connections:
- wire segments 214 -> 217
Changed lines of the file:
@@
 EESchema Schematic File Version 4
-LIBS:sensor_node-cache
-EELAYER 26 0
+EELAYER 30 0
 EELAYER END
 $Descr A3 16535 11693
@@
 L Connector:Conn_Coaxial ANT1
 U 1 1 5C2A1AEB
-P 4350 8450
-F 0 "ANT1" H 4449 8426 50  0000 L CNN
-F 1 "Conn_Coaxial" H 4449 8335 50  0000 L CNN
-F 2 "Connector_Coaxial:SMA_Amphenol_901-144_Vertical" H 4350 8450 50  0001 C CNN
-F 3 " ~" H 4350 8450 50  0001 C CNN
-F 4 "523-901-144-8RFX" H 4350 8450 50  0001 C CNN "Mouser"
-F 5 "4.15" H 0   0   50  0001 C CNN "Price"
-	1    4350 8450
+P 5550 8700
+F 0 "ANT1" H 5649 8676 50  0000 L CNN
+F 1 "Conn_Coaxial" H 5649 8585 50  0000 L CNN
+F 2 "Connector_Coaxial:SMA_Amphenol_901-144_Vertical" H 5550 8700 50  0001 C CNN
+F 3 " ~" H 5550 8700 50  0001 C CNN
+F 4 "523-901-144-8RFX" H 5550 8700 50  0001 C CNN "Mouser"
+F 5 "4.15" H 1200 250 50  0001 C CNN "Price"
+	1    5550 8700
 	1    0    0    -1
 $EndComp
@@
 L power:GND #PWR032
 U 1 1 5C2A57D2
-P 4350 8700
-F 0 "#PWR032" H 4350 8450 50  0001 C CNN
-F 1 "GND" H 4355 8527 50  0000 C CNN
-F 2 "" H 4350 8700 50  0001 C CNN
-F 3 "" H 4350 8700 50  0001 C CNN
-	1    4350 8700
-	1    0    0    -1
-$EndComp
-Wire Wire Line
-	4350 8700 4350 8650
+P 5550 8900
+F 0 "#PWR032" H 5550 8650 50  0001 C CNN
+F 1 "GND" H 5555 8727 50  0000 C CNN
+F 2 "" H 5550 8900 50  0001 C CNN
+F 3 "" H 5550 8900 50  0001 C CNN
+	1    5550 8900
+	1    0    0    -1
+$EndComp
 Wire Wire Line
 	3600 8450 3700 8450
@@
 F 0 "I2C1" H 13650 2600 50  0000 L CNN
 F 1 "Conn_01x05" H 13550 2500 50  0000 L CNN
-F 2 "Connector_JST:JST_XH_B05B-XH-A_1x05_P2.50mm_Vertical" H 13750 2250 50  0001 C CNN
+F 2 "Connector_JST:JST_XH_B5B-XH-A_1x05_P2.50mm_Vertical" H 13750 2250 50  0001 C CNN
 F 3 "~" H 13750 2250 50  0001 C CNN
 F 4 "Farnell: 1516281" H 0   0   50  0001 C CNN "Mouser"
@@
 NoConn ~ 3600 9150
 Wire Notes Line
-	1500 7550 5150 7550
-Wire Notes Line
 	1500 7550 1500 9900
 Wire Notes Line
-	1500 9900 5150 9900
-Wire Notes Line
-	5150 7550 5150 9900
+	5900 7550 5900 9900
 Text Label 15300 8050 2    50   ~ 0
 RX_SW
@@
 Wire Wire Line
 	14700 8250 15700 8250
-Wire Wire Line
-	3700 8450 4150 8450
 $Comp
 L Device:R R9
@@
 	1900 8100 3000 8100
 NoConn ~ 12300 1150
+$Comp
+L Device:Antenna AE2
+U 1 1 617A861F
+P 5550 8000
+F 0 "AE2" H 5630 7991 50  0000 L CNN
+F 1 "Antenna" H 5630 7900 50  0000 L CNN
+F 2 "RF_Antenna:Texas_SWRA416_868MHz_915MHz" H 5550 8000 50  0001 C CNN
+F 3 "~" H 5550 8000 50  0001 C CNN
+F 4 "0" H 1850 -250 50  0001 C CNN "Price"
+	1    5550 8000
+	1    0    0    -1
+$EndComp
+Wire Notes Line
+	1500 7550 5900 7550
+Wire Notes Line
+	1500 9900 5900 9900
+$Comp
+L Jumper:Jumper_3_Open JP1
+U 1 1 617ED0B6
+P 4850 8450
+F 0 "JP1" V 4804 8537 50  0000 L CNN
+F 1 "Jumper_3_Open" V 4895 8537 50  0000 L CNN
+F 2 "Jumper:SolderJumper-3_P1.3mm_Open_Pad1.0x1.5mm" H 4850 8450 50  0001 C CNN
+F 3 "~" H 4850 8450 50  0001 C CNN
+	1    4850 8450
+	0    1    1    0
+$EndComp
+Wire Wire Line
+	3700 8450 4700 8450
+Wire Wire Line
+	4850 8700 5350 8700
+$Comp
+L Device:C C1
+U 1 1 6184B84F
+P 5050 8200
+F 0 "C1" V 4798 8200 50  0000 C CNN
+F 1 "1pF" V 4889 8200 50  0000 C CNN
+F 2 "Capacitor_SMD:C_0603_1608Metric" H 5088 8050 50  0001 C CNN
+F 3 "~" H 5050 8200 50  0001 C CNN
+	1    5050 8200
+	0    1    1    0
+$EndComp
+$Comp
+L Device:L L2
+U 1 1 6184C250
+P 5300 8050
+F 0 "L2" H 5353 8096 50  0000 L CNN
+F 1 "12nH" H 5353 8005 50  0000 L CNN
+F 2 "Inductor_SMD:L_0603_1608Metric" H 5300 8050 50  0001 C CNN
+F 3 "~" H 5300 8050 50  0001 C CNN
+	1    5300 8050
+	1    0    0    -1
+$EndComp
+Wire Wire Line
+	4850 8200 4900 8200
+Wire Wire Line
+	5200 8200 5300 8200
+Connection ~ 5300 8200
+Wire Wire Line
+	5300 8200 5550 8200
+$Comp
+L power:GND #PWR0105
+U 1 1 61870A66
+P 5300 7900
+F 0 "#PWR0105" H 5300 7650 50  0001 C CNN
+F 1 "GND" H 5305 7727 50  0000 C CNN
+F 2 "" H 5300 7900 50  0001 C CNN
+F 3 "" H 5300 7900 50  0001 C CNN
+	1    5300 7900
+	-1   0    0    1
+$EndComp
 $EndSCHEMATC

Commit message: New routing design.
Parts:
- removed C15: 100nF, Capacitor_SMD:C_0603_1608Metric, symbol Device:C
- removed H7: MountingHole, MountingHole:MountingHole_3.2mm_M3, symbol Mechanical:MountingHole
- removed J1: Conn_02x03_Counter_Clockwise, Connector_PinHeader_2.54mm:PinHeader_2x03_P2.54mm_Vertical, symbol Connector_Generic:Conn_02x03_Counter_Clockwise
- removed J2, J4, J5: Conn_01x02, Connector_PinHeader_2.54mm:PinHeader_1x02_P2.54mm_Vertical, symbol Connector_Generic:Conn_01x02
- removed SPI1, SPI2: Conn_01x06, Connector_JST:JST_XH_B06B-XH-A_1x06_P2.50mm_Vertical, symbol Connector_Generic:Conn_01x06
- removed U5: SHTC3, gems_footprints:DFN_4_Pin_2x2mm, symbol GEMS:SHTC3
- added J2: Conn_02x03_Odd_Even, Connector_PinHeader_2.54mm:PinHeader_2x03_P2.54mm_Vertical, symbol Connector_Generic:Conn_02x03_Odd_Even
- I2C1: footprint Connector_JST:JST_XH_B5B-XH-A_1x05_P2.50mm_Vertical -> gems_footprints:TerminalBlock_Phoenix_PTSA-1,2-2-3,5-F-THR-1x05-P3.50mm_45Degree; Mouser Farnell: 1516281 -> 651-1984992
- I2C2, I2C3: footprint Connector_JST:JST_XH_B05B-XH-A_1x05_P2.50mm_Vertical -> gems_footprints:TerminalBlock_Phoenix_PTSA-1,2-2-3,5-F-THR-1x05-P3.50mm_45Degree; Mouser Farnell: 1516281 -> 651-1984992
- IO2, IO3, OWI1, OWI2: footprint Connector_JST:JST_XH_B03B-XH-A_1x03_P2.50mm_Vertical -> gems_footprints:TerminalBlock_Phoenix_PTSA-1,2-2-3,5-F-THR-1x03-P3.50mm_45Degree; Mouser Farnell: 1516277 -> 651-1984976
- IO4: value BOOT OPTION -> BOOT
Connections:
- net labels removed: D1, DAC, ~CS1, ~CS2
- wire segments 217 -> 184
- no-connect marks 15 -> 20
Other:
- note removed: "I2C devives"

Commit message: Add Mouser order codes.
Parts:
- C1: Mouser (none) -> 603-CC603BRNPO9BN1R0
- L2: Mouser (none) -> 81-LQW18AN12NG80D
Changed lines of the file:
@@
 F 2 "Capacitor_SMD:C_0603_1608Metric" H 5088 8050 50  0001 C CNN
 F 3 "~" H 5050 8200 50  0001 C CNN
+F 4 "603-CC603BRNPO9BN1R0" H 5050 8200 50  0001 C CNN "Mouser"
 	1    5050 8200
 	0    1    1    0
@@
 F 2 "Inductor_SMD:L_0603_1608Metric" H 5300 8050 50  0001 C CNN
 F 3 "~" H 5300 8050 50  0001 C CNN
+F 4 "81-LQW18AN12NG80D" H 5300 8050 50  0001 C CNN "Mouser"
 	1    5300 8050
 	1    0    0    -1

Commit message: Fix AT.
Parts:
- IC1: value PCF2129AT -> PCF2129T
Changed lines of the file:
@@
 P 1800 1800
 F 0 "IC1" H 1400 2500 50  0000 C CNN
-F 1 "PCF2129AT" H 1650 2400 50  0000 C CNN
+F 1 "PCF2129T" H 1650 2400 50  0000 C CNN
 F 2 "gems_footprints:SO20" H 2950 1900 50  0001 L CNN
 F 3 "https://www.nxp.com/docs/en/data-sheet/PCF2129.pdf" H 2950 1800 50  0001 L CNN
