File: pcb_boards/sensor_node/sensor_node.kicad_sch (KiCad schematic)
At the start: 61 parts

Commit message: New PDB version.
sensor node: added FTDI chip for USB comms
sensor node: implemented page feedback
sensor node: remove aerial, and SMA connector, update interfacing and RTC

sensor hat: update to two PCBs for reduced thermal conductivity
Parts:
- removed AE2: (no value), symbol Device:Antenna
- removed ANT1: (no value), symbol Connector:Conn_Coaxial
- removed I2C1, I2C2, I2C3: (no value), symbol Connector_Generic:Conn_01x05
- removed IC1: (no value), symbol GEMS:PCF2129AT
- removed IO2, IO3, OWI1, OWI2: (no value), symbol Connector_Generic:Conn_01x03
- removed JP1: (no value), symbol sensor_node-rescue:Jumper_3_Open-Jumper
- removed L2: (no value), symbol Device:L
- added D1: LED, LED_SMD:LED_0603_1608Metric, symbol Device:LED
- added FID1, FID2, FID3: Fiducial, Fiducial:Fiducial_1mm_Mask2mm, symbol Mechanical:Fiducial
- added IC1: PCF2129T, gems_footprints:SO16, symbol GEMS:PCF2129T
- added J1: Screw_Terminal_01x15, gems_footprints:TerminalBlock_Phoenix_PTSA-1,2-2-3,5-F-THR-1x15-P3.50mm_45Degree, symbol Connector:Screw_Terminal_01x15
- added J4: Screw_Terminal_01x12, gems_footprints:TerminalBlock_Phoenix_PTSA-1,2-2-3,5-F-THR-1x12-P3.50mm_45Degree, symbol Connector:Screw_Terminal_01x12
- added R6: 750R, Resistor_SMD:R_0603_1608Metric, symbol Device:R
- added U4: FT232RL, Package_SO:SSOP-28_5.3x10.2mm_P0.65mm, symbol pcb_gateway-rescue:FT232RL-Interface_USB
- AE1: value (none) -> Antenna; footprint (none) -> Connector_PinHeader_2.54mm:PinHeader_1x01_P2.54mm_Vertical; Comment (none) -> Wire antenna, to be soldered by user
- BT1: value (none) -> Battery_Cell; footprint (none) -> gems_footprints:Renata_Battery_Holder_SMTM1125; Manufacturer_Part_Number (none) -> SMTM1225; Notes BR-1225/BN -> (none)
- BT2: value (none) -> Battery_Cell; footprint (none) -> Connector_JST:JST_EH_B02B-EH-A_1x02_P2.50mm_Vertical; Manufacturer_Part_Number (none) -> B2B-EH-A(LF)(SN); Mouser 485-1769 -> 2399159
- BT3: value (none) -> Battery_Cell; footprint (none) -> gems_footprints:Eagle_Battery_Holder_A_12BH311P-GR; Farnell battery AA (none) -> 1365937; Manufacturer_Part_Number (none) -> 12BH311P-GR; Mouser Farnell 1365937 -> 12BH311P-GR; Price 9.23 -> (none)
- C1: value (none) -> 100nF; footprint (none) -> Capacitor_SMD:C_0603_1608Metric; Mouser 603-CC603BRNPO9BN1R0 -> 810-CGA3E2X8R1E104K; Price (none) -> 0.136
- C10, C4, C5, C7, C9: value (none) -> 100nF; footprint (none) -> Capacitor_SMD:C_0603_1608Metric; Manufacturer_Part_Number (none) -> CGA3E2X8R1E104K
- C11, C6: value (none) -> 6.8µF; footprint (none) -> Capacitor_SMD:C_1206_3216Metric; Manufacturer_Part_Number (none) -> CGA5L1X7R1C685MC
- C13, C14, C17: value (none) -> 10uF; footprint (none) -> Capacitor_SMD:C_1206_3216Metric; Manufacturer_Part_Number (none) -> TMK325BJ106KM-P
- C16, C18: value (none) -> 22uF; footprint (none) -> Capacitor_SMD:C_1206_3216Metric; Manufacturer_Part_Number (none) -> TMK316BBJ226ML-T
- D2: value (none) -> LED; footprint (none) -> LED_SMD:LED_0603_1608Metric; Manufacturer_Part_Number (none) -> TLMY1000
- D3: value (none) -> D_Schottky; footprint (none) -> Diode_SMD:D_SMB; Manufacturer_Part_Number (none) -> TLMY1000; Mouser 621-B340LB-F -> 78-TLMY1000
- D4: value (none) -> LED; footprint (none) -> LED_SMD:LED_0603_1608Metric; Manufacturer_Part_Number (none) -> TLMY1000; Mouser 78-TLMS1000 -> 78-TLMY1000
- FB1: value (none) -> Ferrite_Bead; footprint (none) -> Inductor_SMD:L_0805_2012Metric_Pad1.15x1.40mm_HandSolder; Manufacturer_Part_Number (none) -> MI0805K400R-10
- H1, H2, H3, H4: value (none) -> MountingHole; footprint (none) -> MountingHole:MountingHole_3.2mm_M3
- IO4: value (none) -> BOOT; footprint (none) -> Button_Switch_SMD:SW_SPST_KMR2; Manufacturer_Part_Number (none) -> KMR621NGLFS
- J2: value (none) -> Conn_02x03_Odd_Even; footprint (none) -> Connector_PinHeader_2.54mm:PinHeader_2x03_P2.54mm_Vertical; Manufacturer_Part_Number (none) -> 944-10-080-00
- J3: value (none) -> USB_B_Micro; footprint (none) -> Connector_USB:USB_Micro-B_Molex-105017-0001; Manufacturer_Part_Number (none) -> 105017-0001
- JP2: value (none) -> Jumper_3_Open; footprint (none) -> Connector_PinHeader_2.54mm:PinHeader_1x03_P2.54mm_Vertical; Manufacturer_Part_Number (none) -> 4-103321-5
- L1: value (none) -> 2.2uH; footprint (none) -> gems_footprints:L_L4mm_D4mm_H1.8mm; Manufacturer_Part_Number (none) -> TYS40182R2M-10
- R1, R14, R15, R2, R4, R5, R8: value (none) -> 10k; footprint (none) -> Resistor_SMD:R_0603_1608Metric; Manufacturer_Part_Number (none) -> APC0603B10K0N
- R10, R12: value (none) -> 4.7k; footprint (none) -> Resistor_SMD:R_0603_1608Metric; Manufacturer_Name (none) -> Vishay; Manufacturer_Part_Number (none) -> CRCW06034K70JNEAC
- R16, R7: value (none) -> 750R; footprint (none) -> Resistor_SMD:R_0603_1608Metric; Manufacturer_Part_Number (none) -> RC0603FR-07750RL
- R3: value (none) -> 330R; footprint (none) -> Resistor_SMD:R_0603_1608Metric; Manufacturer_Part_Number (none) -> RC0603JR-07330RL
- R9: value (none) -> 10M; footprint (none) -> Resistor_SMD:R_0603_1608Metric; Manufacturer_Part_Number (none) -> CRCW060310M0FKEAC
- RESET1: value (none) -> RESET; footprint (none) -> Button_Switch_SMD:SW_SPST_KMR2; Manufacturer_Name (none) -> C&K; Manufacturer_Part_Number (none) -> KMR621NGLFS
- U1, U8: value (none) -> SiP32431; footprint (none) -> Package_TO_SOT_SMD:SOT-363_SC-70-6; Manufacturer_Name (none) -> Vishay; Manufacturer_Part_Number (none) -> SIP32431DR3-T1GE3
- U2: value (none) -> ESP32-WROOM-32; footprint (none) -> RF_Module:ESP32-WROOM-32; Manufacturer_Name (none) -> Espressif Systems; Manufacturer_Part_Number (none) -> ESP32-WROOM-32D-N16
- U3: value (none) -> RF-LORA-868-SO; footprint (none) -> gems_footprints:RF-LORA-868-SMT; Manufacturer_Name (none) -> RF Solutions; Manufacturer_Part_Number (none) -> RF-LORA-868-SO
- U7: value (none) -> RP604x; footprint (none) -> gems_footprints:DFN_12_Pin_2.7x3mm_P0.5mm; Manufacturer_Name (none) -> Nisshinbo; Manufacturer_Part_Number (none) -> RP604K331A-TR
Connections:
- net A1: now also J4.2 (Pin_2)
- net A2: now also J4.5 (Pin_5)
- net BBS: now also IC1.14 (BBS), IC1.5 (IFS)
- net D+: now also U4.15 (USBD+)
- net D-: now also U4.16 (USBD-)
- net GND: now also C1.2, D1.1 (K), IC1.2 (SDI), IC1.8 (VSS), J1.10 (Pin_10), J1.15 (Pin_15), J1.5 (Pin_5), J4.12 (Pin_12), J4.3 (Pin_3), J4.6 (Pin_6), J4.9 (Pin_9), U4.18 (GND), U4.21 (GND), U4.25 (AGND), U4.26 (TEST), U4.7 (GND)
- net INT_T: now also IC1.13 (~{INT})
- net ONE_W1: now also J4.8 (Pin_8)
- net ONE_W2: now also J4.11 (Pin_11)
- net RX: now also U4.5 (RXD)
- net SCL: now also IC1.1 (SCL), J1.12 (Pin_12), J1.2 (Pin_2), J1.7 (Pin_7)
- net SDA: now also IC1.4 (SDA/~{CE}), J1.13 (Pin_13), J1.3 (Pin_3), J1.8 (Pin_8)
- net TX: now also U4.1 (TXD)
- net VBUS: now also U4.20 (VCC)
- net VPP: now also J1.1 (Pin_1), J1.11 (Pin_11), J1.6 (Pin_6), J4.1 (Pin_1), J4.10 (Pin_10), J4.4 (Pin_4), J4.7 (Pin_7)
- net ~{RST_I2C}: now also J1.14 (Pin_14), J1.4 (Pin_4), J1.9 (Pin_9)
- net at BT1.1 (+), C4.2: now also IC1.15 (VBAT)
- net at R3.1: now also IC1.16 (VDD)
- net at C1.1: now also U4.17 (3V3OUT), U4.4 (VCCIO)
- net +3V3 renamed +3.3V
- new net: R6.1, U4.23 (CBUS0)
- new net: D1.2 (A), R6.2
- no-connect marks 20 -> 31
Other:
- moved on the sheet: R10, R12, R4, R5
