File: pcb_boards/radiation_shield/radiation_shield.sch (KiCad schematic (older format))
At the start: 6 parts, among them J1 Conn_01x05, U1 APDS-9306-065, U2 SHT35

Commit message: Update.
Parts:
- C1: Mouser (none) -> 710-885012206083; Price (none) -> 0.085
- C2: Mouser (none) -> 810-CGA3E2X8R1E104K; Price (none) -> 0.136
- J1: Mouser (none) -> Farnell: 1516281; Price (none) -> 0.138
- R1: Mouser (none) -> 284-APC0603B10K0N; Price (none) -> 0.102
- U1: Mouser (none) -> 630-APDS-9306-065; Price (none) -> 0.983
- U2: Mouser (none) -> 403-SHT35-DIS-F; Price (none) -> 8.16
Changed lines of the file:
@@
 EESchema Schematic File Version 4
-LIBS:light_sensor-cache
+LIBS:radiation_shield-cache
 EELAYER 26 0
 EELAYER END
@@
 F 2 "gems_footprints:APDS-9306-065" H 1850 2350 50  0001 C CNN
 F 3 "https://www.mouser.com/datasheet/2/678/V02-4755EN_DS_APDS-9306_2016-10-21-1130983.pdf" H 1850 2350 50  0001 C CNN
+F 4 "630-APDS-9306-065" H 0   0   50  0001 C CNN "Mouser"
+F 5 "0.983" H 0   0   50  0001 C CNN "Price"
 	1    1850 2350
 	1    0    0    -1
@@
 F 2 "Connector_JST:JST_XH_B05B-XH-A_1x05_P2.50mm_Vertical" H 7750 2250 50  0001 C CNN
 F 3 "~" H 7750 2250 50  0001 C CNN
+F 4 "Farnell: 1516281" H 0   0   50  0001 C CNN "Mouser"
+F 5 "0.138" H 0   0   50  0001 C CNN "Price"
 	1    7750 2250
 	1    0    0    -1
@@
 F 2 "Capacitor_SMD:C_0603_1608Metric" H 1288 2500 50  0001 C CNN
 F 3 "~" H 1250 2650 50  0001 C CNN
+F 4 "710-885012206083" H 0   0   50  0001 C CNN "Mouser"
+F 5 "0.085" H 0   0   50  0001 C CNN "Price"
 	1    1250 2650
 	1    0    0    -1
@@
 F 2 "gems_footprints:8P-1EP-DFN_2.5x2.5" H 4550 2300 50  0001 C CNN
 F 3 "https://www.sensirion.com/fileadmin/user_upload/customers/sensirion/Dokumente/0_Datasheets/Humidity/Sensirion_Humidity_Sensors_SHT3x_Datasheet_digital.pdf" H 4550 2300 50  0001 C CNN
+F 4 "403-SHT35-DIS-F" H 4550 2300 50  0001 C CNN "Mouser"
+F 5 "8.16" H 4550 2300 50  0001 C CNN "Price"
 	1    4550 2300
 	1    0    0    -1
@@
 F 2 "Capacitor_SMD:C_0603_1608Metric" H 6038 2100 50  0001 C CNN
 F 3 "~" H 6000 2250 50  0001 C CNN
+F 4 "810-CGA3E2X8R1E104K" H 0   0   50  0001 C CNN "Mouser"
+F 5 "0.136" H 0   0   50  0001 C CNN "Price"
 	1    6000 2250
 	1    0    0    -1
@@
 F 2 "Resistor_SMD:R_0603_1608Metric" V 6480 2250 50  0001 C CNN
 F 3 "~" H 6550 2250 50  0001 C CNN
+F 4 "284-APC0603B10K0N" H 0   0   50  0001 C CNN "Mouser"
+F 5 "0.102" H 0   0   50  0001 C CNN "Price"
 	1    6550 2250
 	1    0    0    -1

Commit message: Update.
Connections:
- wire segments 19 -> 21
- no-connect marks 3 -> 2
Changed lines of the file:
@@
 EESchema Schematic File Version 4
-LIBS:radiation_shield-cache
-EELAYER 26 0
+EELAYER 30 0
 EELAYER END
 $Descr A4 11693 8268
@@
 	-1   0    0    1
 $EndComp
+Text Label 5550 2250 2    50   ~ 0
+SCL
+Text Label 5550 2400 2    50   ~ 0
+SDA
+NoConn ~ 3900 2250
+Wire Wire Line
+	7350 2350 7550 2350
+Text Label 7350 2350 0    50   ~ 0
+~RST
+Text Label 3650 2100 0    50   ~ 0
+~RST
+Wire Wire Line
+	3650 2100 3900 2100
+Wire Wire Line
+	5550 2250 5200 2250
+Wire Wire Line
+	5550 2400 5200 2400
+Wire Wire Line
+	4550 2850 3900 2850
+$Comp
+L power:GND #PWR03
+U 1 1 5D31E046
+P 4550 2850
+F 0 "#PWR03" H 4550 2600 50  0001 C CNN
+F 1 "GND" H 4555 2677 50  0000 C CNN
+F 2 "" H 4550 2850 50  0001 C CNN
+F 3 "" H 4550 2850 50  0001 C CNN
+	1    4550 2850
+	1    0    0    -1
+$EndComp
+$Comp
+L power:+3.3V #PWR06
+U 1 1 5D31E28E
+P 5550 2100
+F 0 "#PWR06" H 5550 1950 50  0001 C CNN
+F 1 "+3.3V" H 5565 2273 50  0000 C CNN
+F 2 "" H 5550 2100 50  0001 C CNN
+F 3 "" H 5550 2100 50  0001 C CNN
+	1    5550 2100
+	1    0    0    -1
+$EndComp
+Wire Wire Line
+	5550 2100 5200 2100
+$Comp
+L Device:C C2
+U 1 1 5D31EB78
+P 6000 2250
+F 0 "C2" H 6115 2296 50  0000 L CNN
+F 1 "0.1uF" H 6115 2205 50  0000 L CNN
+F 2 "Capacitor_SMD:C_0603_1608Metric" H 6038 2100 50  0001 C CNN
+F 3 "~" H 6000 2250 50  0001 C CNN
+F 4 "810-CGA3E2X8R1E104K" H 0   0   50  0001 C CNN "Mouser"
+F 5 "0.136" H 0   0   50  0001 C CNN "Price"
+	1    6000 2250
+	1    0    0    -1
+$EndComp
+$Comp
+L power:+3.3V #PWR07
+U 1 1 5D31EBA4
+P 6000 2100
+F 0 "#PWR07" H 6000 1950 50  0001 C CNN
+F 1 "+3.3V" H 6015 2273 50  0000 C CNN
+F 2 "" H 6000 2100 50  0001 C CNN
+F 3 "" H 6000 2100 50  0001 C CNN
+	1    6000 2100
+	1    0    0    -1
+$EndComp
+$Comp
+L power:GND #PWR08
+U 1 1 5D31EBB9
+P 6000 2400
+F 0 "#PWR08" H 6000 2150 50  0001 C CNN
+F 1 "GND" H 6005 2227 50  0000 C CNN
+F 2 "" H 6000 2400 50  0001 C CNN
+F 3 "" H 6000 2400 50  0001 C CNN
+	1    6000 2400
+	1    0    0    -1
+$EndComp
+$Comp
+L Device:R R1
+U 1 1 5D31F19D
+P 6550 2250
+F 0 "R1" H 6620 2296 50  0000 L CNN
+F 1 "10k" H 6620 2205 50  0000 L CNN
+F 2 "Resistor_SMD:R_0603_1608Metric" V 6480 2250 50  0001 C CNN
+F 3 "~" H 6550 2250 50  0001 C CNN
+F 4 "284-APC0603B10K0N" H 0   0   50  0001 C CNN "Mouser"
+F 5 "0.102" H 0   0   50  0001 C CNN "Price"
+	1    6550 2250
+	1    0    0    -1
+$EndComp
+$Comp
+L power:+3.3V #PWR09
+U 1 1 5D31F209
+P 6550 2100
+F 0 "#PWR09" H 6550 1950 50  0001 C CNN
+F 1 "+3.3V" H 6565 2273 50  0000 C CNN
+F 2 "" H 6550 2100 50  0001 C CNN
+F 3 "" H 6550 2100 50  0001 C CNN
+	1    6550 2100
+	1    0    0    -1
+$EndComp
+$Comp
+L power:+3.3V #PWR010
+U 1 1 5D31F227
+P 7350 2050
+F 0 "#PWR010" H 7350 1900 50  0001 C CNN
+F 1 "+3.3V" H 7365 2223 50  0000 C CNN
+F 2 "" H 7350 2050 50  0001 C CNN
+F 3 "" H 7350 2050 50  0001 C CNN
+	1    7350 2050
+	1    0    0    -1
+$EndComp
+Wire Wire Line
+	7350 2450 7550 2450
+Text Label 6800 2500 2    50   ~ 0
+~RST
+Wire Wire Line
+	6800 2500 6550 2500
+Wire Wire Line
+	6550 2500 6550 2400
+Connection ~ 4550 2850
+Wire Wire Line
+	3900 2550 3900 2850
+Wire Wire Line
+	3900 2400 3900 2550
+Connection ~ 3900 2550
 $Comp
 L GEMS:SHT35 U2
@@
 	1    0    0    -1
 $EndComp
-Text Label 5550 2250 2    50   ~ 0
-SCL
-Text Label 5550 2400 2    50   ~ 0
-SDA
-NoConn ~ 5200 2550
-NoConn ~ 3900 2250
-Wire Wire Line
-	7350 2350 7550 2350
-Text Label 7350 2350 0    50   ~ 0
-~RST
-Text Label 3650 2100 0    50   ~ 0
-~RST
-Wire Wire Line
-	3650 2100 3900 2100
-Wire Wire Line
-	5550 2250 5200 2250
-Wire Wire Line
-	5550 2400 5200 2400
-Wire Wire Line
-	4550 2850 3900 2850
-Wire Wire Line
-	3900 2550 3900 2850
-$Comp
-L power:GND #PWR03
-U 1 1 5D31E046
-P 4550 2850
-F 0 "#PWR03" H 4550 2600 50  0001 C CNN
-F 1 "GND" H 4555 2677 50  0000 C CNN
-F 2 "" H 4550 2850 50  0001 C CNN
-F 3 "" H 4550 2850 50  0001 C CNN
-	1    4550 2850
-	1    0    0    -1
-$EndComp
-Connection ~ 4550 2850
-Wire Wire Line
-	3900 2400 3900 2550
-Connection ~ 3900 2550
-$Comp
-L power:+3.3V #PWR06
-U 1 1 5D31E28E
-P 5550 2100
-F 0 "#PWR06" H 5550 1950 50  0001 C CNN
-F 1 "+3.3V" H 5565 2273 50  0000 C CNN
-F 2 "" H 5550 2100 50  0001 C CNN
-F 3 "" H 5550 2100 50  0001 C CNN
-	1    5550 2100
-	1    0    0    -1
-$EndComp
-Wire Wire Line
-	5550 2100 5200 2100
-$Comp
-L Device:C C2
-U 1 1 5D31EB78
-P 6000 2250
-F 0 "C2" H 6115 2296 50  0000 L CNN
-F 1 "0.1uF" H 6115 2205 50  0000 L CNN
-F 2 "Capacitor_SMD:C_0603_1608Metric" H 6038 2100 50  0001 C CNN
-F 3 "~" H 6000 2250 50  0001 C CNN
-F 4 "810-CGA3E2X8R1E104K" H 0   0   50  0001 C CNN "Mouser"
-F 5 "0.136" H 0   0   50  0001 C CNN "Price"
-	1    6000 2250
-	1    0    0    -1
-$EndComp
-$Comp
-L power:+3.3V #PWR07
-U 1 1 5D31EBA4
-P 6000 2100
-F 0 "#PWR07" H 6000 1950 50  0001 C CNN
-F 1 "+3.3V" H 6015 2273 50  0000 C CNN
-F 2 "" H 6000 2100 50  0001 C CNN
-F 3 "" H 6000 2100 50  0001 C CNN
-	1    6000 2100
-	1    0    0    -1
-$EndComp
-$Comp
-L power:GND #PWR08
-U 1 1 5D31EBB9
-P 6000 2400
-F 0 "#PWR08" H 6000 2150 50  0001 C CNN
-F 1 "GND" H 6005 2227 50  0000 C CNN
-F 2 "" H 6000 2400 50  0001 C CNN
-F 3 "" H 6000 2400 50  0001 C CNN
-	1    6000 2400
-	1    0    0    -1
-$EndComp
-$Comp
-L Device:R R1
-U 1 1 5D31F19D
-P 6550 2250
-F 0 "R1" H 6620 2296 50  0000 L CNN
-F 1 "10k" H 6620 2205 50  0000 L CNN
-F 2 "Resistor_SMD:R_0603_1608Metric" V 6480 2250 50  0001 C CNN
-F 3 "~" H 6550 2250 50  0001 C CNN
-F 4 "284-APC0603B10K0N" H 0   0   50  0001 C CNN "Mouser"
-F 5 "0.102" H 0   0   50  0001 C CNN "Price"
-	1    6550 2250
-	1    0    0    -1
-$EndComp
-$Comp
-L power:+3.3V #PWR09
-U 1 1 5D31F209
-P 6550 2100
-F 0 "#PWR09" H 6550 1950 50  0001 C CNN
-F 1 "+3.3V" H 6565 2273 50  0000 C CNN
-F 2 "" H 6550 2100 50  0001 C CNN
-F 3 "" H 6550 2100 50  0001 C CNN
-	1    6550 2100
-	1    0    0    -1
-$EndComp
-$Comp
-L power:+3.3V #PWR010
-U 1 1 5D31F227
-P 7350 2050
-F 0 "#PWR010" H 7350 1900 50  0001 C CNN
-F 1 "+3.3V" H 7365 2223 50  0000 C CNN
-F 2 "" H 7350 2050 50  0001 C CNN
-F 3 "" H 7350 2050 50  0001 C CNN
-	1    7350 2050
-	1    0    0    -1
-$EndComp
-Wire Wire Line
-	7350 2450 7550 2450
-Text Label 6800 2500 2    50   ~ 0
-~RST
-Wire Wire Line
-	6800 2500 6550 2500
-Wire Wire Line
-	6550 2500 6550 2400
+Wire Wire Line
+	4550 2850 5200 2850
+Wire Wire Line
+	5200 2850 5200 2550
 $EndSCHEMATC
