File: pcb_boards/radiation_shield/radiation_shield.kicad_pcb (KiCad board)
At the start: 2 copper layers, 30 x 30 mm, 6 parts, among them J1 Conn_01x05, U1 APDS-9306-065, U2 SHT35

Commit message: Update.
Parts:
- moved C2 8.35 mm to (104.4, 97.2), turned to 0 degrees
- moved U2 8.11 mm to (100.4, 99.4)
- moved R1 7.85 mm to (103.6, 99.6)
- moved C1 5.20 mm to (100.0, 109.6)
- turned U1 to 90 degrees
Connections:
- U2 pad 7: Net-(U2-Pad7) -> GND
Routing:
- net /SDA: track 30.0 -> 23.2 mm, vias 2 -> 1
- net +3V3: track 31.1 -> 36.6 mm
- net /SCL: track 21.7 -> 16.9 mm
- net /~RST: track 21.6 -> 17.4 mm
- net GND: track 6.13 -> 8.16 mm, vias 1 -> 8
Other:
- outline, holes or cut-outs redrawn
- board text added: "3.3V"
- board text added: "GND"
- board text added: "Rev. 2"
- board text added: "SCL"
- board text added: "SDA"
- board text added: "sensor hat"
- board text added: "~RST"
- board text removed: "GEMS sensor board"
- board text removed: "Rev. 1"
- board text removed: "light sensor"

Commit message: New PDB version.
sensor node: added FTDI chip for USB comms
sensor node: implemented page feedback
sensor node: remove aerial, and SMA connector, update interfacing and RTC

sensor hat: update to two PCBs for reduced thermal conductivity
Connections:
- net /~RST renamed /~{RST}
Other:
- net class Default removed
- board text added: "~{RST}"
- board text removed: "~RST"
